Commit message: Update servo_gazebo.urdf.xacro

File: servo_hardware_moveit_config/config/servo_gazebo.urdf.xacro (robot description, xacro)
@@ -4,20 +4,10 @@
     <xacro:include filename="$(find servo_hardware)/urdf/servo.description.xacro" />
     <!-- Import servo ros2_control description -->
-    <ros2_control name="GazeboSimSystem" type="system">
-        <hardware>
-            <plugin>gazebo_ros2_control/GazeboSystem</plugin>
-        </hardware>
-        <joint name="servo_joint">
-            <command_interface name="position">
-                <param name="min">-15</param>
-                <param name="max">15</param>
-            </command_interface>
-            <state_interface name="position">
-                <param name="initial_value">1.0</param>
-            </state_interface>
-            <state_interface name="velocity"/>
-            <state_interface name="effort"/>
-        </joint>
-    </ros2_control>
+    <xacro:include filename="servo.ros2_control.xacro" />
+    <xacro:servo_ros2_control
+        name="servo"
+        plugin="gazebo_ros2_control/GazeboSystem"
+        prefix=""
+    />
     <!-- Gazebo Colors & Plugins -->
     <gazebo reference="motor">
